Commit message: collsion mesh 경로 수정

File: src/QUB_urdf/urdf/QUB v1.2_@Mac.urdf (robot description, URDF)
Before this commit: robot QUB, 14 links, 13 joints
Links:
- link base_link: geometry collision box size=0.140 0.200 0.279; visual mesh filename=file:///Users/jae/Library/Mobile Documents/com~apple~CloudD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
- link pelvis_link: geometry collision box size=0.140 0.1194 0.175; visual mesh filename=file:///Users/jae/Library/Mobile Documents/com~apple~CloudD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

Commit message: 오류 확인

File: src/QUB_urdf/urdf/QUB v1.2_@Mac.urdf (robot description, URDF)
Before this commit: robot QUB, 14 links, 13 joints
Links:
- link pelvis_link: geometry collision mesh filename=file:///Users/jae/Library/Mobile Documents/com~apple~CloudD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; visual mesh filename=file:///Users/jae/Library/Mobile Documents/com~apple~CloudD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
